File: Arduino Uno A4988 Shield/_autosave-Arduino Uno A4988 Shield.kicad_pcb (KiCad board)
At the start: 2 copper layers, 68.6 x 53.3 mm, 8 parts, among them J1 Power, J2 Digital/PWM, J3 Analog, J4 Digital/PWM

Commit message: added template
Parts:
- added A1: Pololu_Breakout_A4988, Module:Pololu_Breakout-16_15.2x20.3mm, F.Cu at (126.1, 80.3)
- added J5: Conn_01x04, Connector_PinHeader_2.54mm:PinHeader_1x04_P2.54mm_Vertical, F.Cu at (130.9, 86.5)
