File: Shao Rong Shield/Shao Rong Shield.kicad_pcb (KiCad board)
At the start: 2 copper layers, 68.6 x 53.3 mm, 8 parts, among them J1 Power, J2 Digital/PWM, J3 Analog, J4 Digital/PWM

Commit message: First prototype
Parts:
- added J10: VIBRATION MOTOR, Connector_JST:JST_XH_B3B-XH-A_1x03_P2.50mm_Vertical, F.Cu at (139.5, 60.5)
- added J11: SPARE1, Connector_JST:JST_XH_B3B-XH-A_1x03_P2.50mm_Vertical, F.Cu at (147.5, 74.0)
- added J12: SPARE2, Connector_JST:JST_XH_B3B-XH-A_1x03_P2.50mm_Vertical, F.Cu at (156.5, 83.0)
- added J5: POWER SUPPLY, Connector_JST:JST_XH_S2B-XH-A_1x02_P2.50mm_Horizontal, F.Cu at (103.5, 60.8)
- added J6: STEPPER MOTOR, Connector_JST:JST_XH_B6B-XH-A_1x06_P2.50mm_Vertical, F.Cu at (114.0, 60.5)
- added J7: KEYBOARD, Connector_JST:JST_XH_B3B-XH-A_1x03_P2.50mm_Vertical, F.Cu at (129.0, 60.5)
- added J8: LCD, Connector_JST:JST_XH_B4B-XH-A_1x04_P2.50mm_Vertical, F.Cu at (129.0, 77.5)
- added J9: RS232, Connector_JST:JST_XH_B3B-XH-A_1x03_P2.50mm_Vertical, F.Cu at (159.5, 63.0)
Connections:
- net /SDA/A4 renamed /SDA
- J1 pad 5: +5V -> unconnected-(J1-Pin_5-Pad5)
