File: Shao Rong Shield/Shao Rong Shield.kicad_sch (KiCad schematic)
At the start: 4 parts, among them J1 Power, J2 Digital/PWM, J3 Analog, J4 Digital/PWM

Commit message: First prototype
Parts:
- added J10: VIBRATION MOTOR, Connector_JST:JST_XH_B3B-XH-A_1x03_P2.50mm_Vertical, symbol Connector_Generic:Conn_01x03
- added J11: SPARE1, Connector_JST:JST_XH_B3B-XH-A_1x03_P2.50mm_Vertical, symbol Connector_Generic:Conn_01x03
- added J12: SPARE2, Connector_JST:JST_XH_B3B-XH-A_1x03_P2.50mm_Vertical, symbol Connector_Generic:Conn_01x03
- added J5: POWER SUPPLY, Connector_JST:JST_XH_S2B-XH-A_1x02_P2.50mm_Horizontal, symbol Connector_Generic:Conn_01x02
- added J6: STEPPER MOTOR, Connector_JST:JST_XH_B6B-XH-A_1x06_P2.50mm_Vertical, symbol Connector_Generic:Conn_01x06
- added J7: KEYBOARD, Connector_JST:JST_XH_B3B-XH-A_1x03_P2.50mm_Vertical, symbol Connector_Generic:Conn_01x03
- added J8: LCD, Connector_JST:JST_XH_B4B-XH-A_1x04_P2.50mm_Vertical, symbol Connector_Generic:Conn_01x04
- added J9: RS232, Connector_JST:JST_XH_B3B-XH-A_1x03_P2.50mm_Vertical, symbol Connector_Generic:Conn_01x03
Connections:
- net *10: now also J9.2 (Pin_2)
- net *11: now also J9.3 (Pin_3)
- net *5: now also J11.3 (Pin_3)
- net *6: now also J10.3 (Pin_3)
- net *9: now also J6.5 (Pin_5)
- net +5V: now also J10.1 (Pin_1), J11.1 (Pin_1), J12.1 (Pin_1), J5.1 (Pin_1), J6.1 (Pin_1), J7.1 (Pin_1), J8.1 (Pin_1); no longer J1.5 (Pin_5)
- net 12: now also J6.4 (Pin_4)
- net 13: now also J6.3 (Pin_3)
- net 8: now also J6.6 (Pin_6)
- net A1: now also J7.3 (Pin_3)
- net A2: now also J12.3 (Pin_3)
- net GND: now also J10.2 (Pin_2), J11.2 (Pin_2), J12.2 (Pin_2), J5.2 (Pin_2), J6.2 (Pin_2), J7.2 (Pin_2), J8.2 (Pin_2), J9.1 (Pin_1)
- net SCL/A5: now also J8.4 (Pin_4)
- net SDA/A4 renamed SDA
- net SDA: now also J8.3 (Pin_3)
